File: WorkshopDS1/WorkShopDS1.sch (KiCad schematic (older format))
At the start: 40 parts, among them J1 JACK-DC, J2 TRIGGER INPUT, J3 OUTPUT, SW1 SPDT_small, U1 7414, U2 LM358, U3 LM7805

Commit message: got rid of extra parts - changed a few footprints
Parts:
- removed C1: 100uF, 4ms-footprints:Cap_Electrolytic_TH, symbol CAP-ELEC-TH
- removed C3: 10uF, 4ms-footprints:Cap_Electrolytic_TH, symbol CAP-ELEC-TH
- removed C4: 10uF, 4ms-footprints:Cap_Ceramic_TH, symbol CAP_TH
- removed C5, C6, C8: TBD, 4ms-footprints:Cap_Electrolytic_TH, symbol CAP-ELEC-TH
- removed OSC2POT1: TBD, symbol POT
- removed OSC2SW1: TBD, symbol SPDT_small
- removed R7, R8, R9: TBD, 4ms-footprints:Resistor_TH_300, symbol RTH
- removed U3: LM7805, symbol LM7805
- removed VOLUME1: A500k, symbol POT
- J1: value JACK-DC -> 9v battery; symbol JACK-DC -> 9v_Battery_Clip
- R3: value 470 -> 1k
Connections:
- net +5V is gone; now on net +9V: LATCHING1.2, MOMENTARY1.2, U2.8 (V+), U2.8 (V+)
- net GND: now also R11.1; no longer R11.2
- net at J2.1 (V), SENSE/STARVE1.1 (Left): now also R2.1; no longer R2.2
- net at LATCHING1.1, MOMENTARY1.3: now also R2.2; no longer R2.1
- net +9V: now reaches D1.1 (K)
- net at MOMENTARY3.2: now also C9.2
- net at LED2.2 (C): now also R11.2; no longer R11.1
Other:
- note removed: "BLEND POT BETWEEN OSCILLATORS???"
- note removed: "POWER CIRCUIT\n-NEED TO ADD 9V BATTERY CLIP"
- note removed: "SEPERATE VOLTAGE STARVE FOR LATCHING SWITCH ON?"
- moved on the sheet: C2, C9, D1, J3, LATCHING1, LED2, MOMENTARY1, R10, R11, R2, SW1, U1B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

Commit message: forgot to save
Parts:
- J1, J2, LATCHING1, MOMENTARY1: footprint (none) -> zfoot:Jack_DC
- J3: footprint (none) -> zfoot:Jack_Instrument
- LED2: footprint LED-T1 -> zfoot:Jack_DC
- PITCH1, SENSE/STARVE1: footprint (none) -> zfoot:Jack_Instrument_exp
- U1: footprint (none) -> 4ms-footprints:DIP-14_W7.62mm
- U2: footprint (none) -> 4ms-footprints:DIP_8pin_TL072_TH
Other:
- moved on the sheet: U1B, U1C, U1D
Changed lines of the file:
@@
 F 0 "J2" H 1600 2450 60  0000 C CNN
 F 1 "TRIGGER INPUT" H 1600 2344 60  0000 C CNN
-F 2 "" H 1450 2100 60  0000 C CNN
+F 2 "zfoot:Jack_DC" H 1450 2100 60  0000 C CNN
 F 3 "" H 1450 2100 60  0000 C CNN
 	1    1450 2100
@@
 F 0 "J3" H 7050 3050 60  0000 C CNN
 F 1 "OUTPUT" H 7050 2944 60  0000 C CNN
-F 2 "" H 6900 2700 60  0000 C CNN
+F 2 "zfoot:Jack_Instrument" H 6900 2700 60  0000 C CNN
 F 3 "" H 6900 2700 60  0000 C CNN
 	1    6900 2700
@@
 F 0 "LATCHING1" V 1400 1250 60  0000 L CNN
 F 1 "SPDT_small" V 1453 1838 20  0000 L CNN
-F 2 "" H 1400 1700 60  0001 C CNN
+F 2 "zfoot:Jack_DC" H 1400 1700 60  0001 C CNN
 F 3 "" H 1400 1700 60  0001 C CNN
 	1    1400 1700
@@
 F 0 "MOMENTARY1" V 1400 1550 60  0000 L CNN
 F 1 "SPDT_small" V 1453 1637 20  0000 L CNN
-F 2 "" H 1400 1500 60  0001 C CNN
+F 2 "zfoot:Jack_DC" H 1400 1500 60  0001 C CNN
 F 3 "" H 1400 1500 60  0001 C CNN
 	1    1400 1500
@@
 F 0 "J1" H 1600 4950 60  0000 C CNN
 F 1 "9v battery" H 1600 4844 60  0000 C CNN
-F 2 "" H 1450 4600 60  0000 C CNN
+F 2 "zfoot:Jack_DC" H 1450 4600 60  0000 C CNN
 F 3 "" H 1450 4600 60  0000 C CNN
 	1    1450 4600
@@
 F 0 "SENSE/STARVE1" H 1930 2196 50  0000 R CNN
 F 1 "A50k" H 1930 2105 50  0000 R CNN
-F 2 "" H 2200 1900 50  0001 C CNN
+F 2 "zfoot:Jack_Instrument_exp" H 2200 1900 50  0001 C CNN
 F 3 "" H 2000 2150 50  0001 C CNN
 	1    2000 2150
@@
 F 0 "U2" H 2841 2296 50  0000 L CNN
 F 1 "LM358" H 2841 2205 50  0000 L CNN
-F 2 "" H 2500 2250 50  0001 C CNN
+F 2 "4ms-footprints:DIP_8pin_TL072_TH" H 2500 2250 50  0001 C CNN
 F 3 "" H 2500 2250 50  0001 C CNN
 	1    2500 2250
@@
 F 0 "U2" H 4641 2396 50  0000 L CNN
 F 1 "LM358" H 4641 2305 50  0000 L CNN
-F 2 "" H 4300 2350 50  0001 C CNN
+F 2 "4ms-footprints:DIP_8pin_TL072_TH" H 4300 2350 50  0001 C CNN
 F 3 "" H 4300 2350 50  0001 C CNN
 	2    4300 2350
@@
 F 0 "U1" H 4750 3150 60  0000 L CNN
 F 1 "7414" H 4750 3250 25  0000 L CNN
-F 2 "" H 4600 3700 60  0001 C CNN
+F 2 "4ms-footprints:DIP-14_W7.62mm" H 4600 3700 60  0001 C CNN
 F 3 "" H 4600 3700 60  0001 C CNN
 	1    4650 3050
@@
 F 0 "PITCH1" V 4986 3400 50  0000 C CNN
 F 1 "B50k" V 4895 3400 50  0000 C CNN
-F 2 "" H 5300 3150 50  0001 C CNN
+F 2 "zfoot:Jack_Instrument_exp" H 5300 3150 50  0001 C CNN
 F 3 "" H 5100 3400 50  0001 C CNN
 	1    5100 3400
@@
 L HEX_INV_TRI_DirPwr U1
 U 2 1 5A1D5267
-P 4950 1150
-F 0 "U1" H 5050 1250 60  0000 L CNN
-F 1 "7414" H 5050 1350 25  0000 L CNN
-F 2 "" H 4900 1800 60  0001 C CNN
-F 3 "" H 4900 1800 60  0001 C CNN
-	2    4950 1150
+P 4700 1150
+F 0 "U1" H 4800 1250 60  0000 L CNN
+F 1 "7414" H 4800 1350 25  0000 L CNN
+F 2 "4ms-footprints:DIP-14_W7.62mm" H 4650 1800 60  0001 C CNN
+F 3 "" H 4650 1800 60  0001 C CNN
+	2    4700 1150
 	1    0    0    -1
 $EndComp
@@
 L HEX_INV_TRI_DirPwr U1
 U 3 1 5A1D54FF
-P 5650 1150
-F 0 "U1" H 5750 1250 60  0000 L CNN
-F 1 "7414" H 5750 1350 25  0000 L CNN
-F 2 "" H 5600 1800 60  0001 C CNN
-F 3 "" H 5600 1800 60  0001 C CNN
-	3    5650 1150
+P 5500 1150
+F 0 "U1" H 5600 1250 60  0000 L CNN
+F 1 "7414" H 5600 1350 25  0000 L CNN
+F 2 "4ms-footprints:DIP-14_W7.62mm" H 5450 1800 60  0001 C CNN
+F 3 "" H 5450 1800 60  0001 C CNN
+	3    5500 1150
 	1    0    0    -1
 $EndComp
@@
 L HEX_INV_TRI_DirPwr U1
 U 4 1 5A1D5561
-P 6400 1150
-F 0 "U1" H 6500 1250 60  0000 L CNN
-F 1 "7414" H 6500 1350 25  0000 L CNN
-F 2 "" H 6350 1800 60  0001 C CNN
-F 3 "" H 6350 1800 60  0001 C CNN
-	4    6400 1150
+P 6200 1150
+F 0 "U1" H 6300 1250 60  0000 L CNN
+F 1 "7414" H 6300 1350 25  0000 L CNN
+F 2 "4ms-footprints:DIP-14_W7.62mm" H 6150 1800 60  0001 C CNN
+F 3 "" H 6150 1800 60  0001 C CNN
+	4    6200 1150
 	1    0    0    -1
 $EndComp
@@
 F 0 "U1" H 2100 3300 60  0000 L CNN
 F 1 "7414" H 2100 3400 25  0000 L CNN
-F 2 "" H 1950 3850 60  0001 C CNN
+F 2 "4ms-footprints:DIP-14_W7.62mm" H 1950 3850 60  0001 C CNN
 F 3 "" H 1950 3850 60  0001 C CNN
 	6    2000 3200
@@
 F 0 "LED2" H 2400 4446 45  0000 C CNN
 F 1 "LED" H 2400 4530 45  0000 C CNN
-F 2 "LED-T1" H 2380 4800 20  0001 C CNN
+F 2 "zfoot:Jack_DC" H 2380 4800 20  0001 C CNN
 F 3 "" H 2350 4650 60  0001 C CNN
 	1    2350 4650
@@
 F 0 "U1" H 7150 1250 60  0000 L CNN
 F 1 "7414" H 7150 1350 25  0000 L CNN
-F 2 "" H 7000 1800 60  0001 C CNN
+F 2 "4ms-footprints:DIP-14_W7.62mm" H 7000 1800 60  0001 C CNN
 F 3 "" H 7000 1800 60  0001 C CNN
 	5    7050 1150
