File: DS8/DS8.sch (KiCad schematic (older format))
At the start: 101 parts, among them P1 CONN-02x05, Q1 3904, Q2 3904, U0 LM13700, U1 LM385, U2 LM385, U3 LM385, U4 LM385, U5 LM385, U6 KA78L05

Commit message: built up the board - works but needs tweaking!
Parts:
- C1: value 3.3uF - 10uF on proto -> 2.2uF
- C11: value 0.1uF -> 10nF - CONTROLS PITCH
- C3: value 3.3uF - 10uF on proto -> OMITTED SUPPOSED TO BE 3.3
- C6: value 22pF -> 1nF get rid of shitty high pitch noise
Changed lines of the file:
@@
 AR Path="/5DCE035A/5E16E6E0" Ref="C?"  Part="1"
 F 0 "C1" H 3800 1675 50  0000 L CNN
-F 1 "3.3uF - 10uF on proto" H 3725 1750 50  0000 L CNN
+F 1 "2.2uF" H 3725 1750 50  0000 L CNN
 F 2 "4ms_Capacitor:C_0805" H 3700 1675 50  0001 C CNN
 F 3 "" H 3700 1675 50  0000 C CNN
@@
 AR Path="/5DCE035A/5E286DAB" Ref="C?"  Part="1"
 F 0 "C3" H 6150 2050 50  0000 L CNN
-F 1 "3.3uF - 10uF on proto" H 6075 2125 50  0000 L CNN
+F 1 "OMITTED SUPPOSED TO BE 3.3" H 6075 2125 50  0000 L CNN
 F 2 "4ms_Capacitor:C_0805" H 6050 2050 50  0001 C CNN
 F 3 "" H 6050 2050 50  0000 C CNN
@@
 AR Path="/5DCE035A/5E9B7779" Ref="C?"  Part="1"
 F 0 "C11" H 6250 5725 50  0000 L CNN
-F 1 "0.1uF" H 6175 5650 50  0000 L CNN
+F 1 "10nF - CONTROLS PITCH" V 7150 5350 50  0000 L CNN
 F 2 "4ms_Capacitor:C_0603" H 6450 5675 50  0001 C CNN
 F 3 "" H 6450 5675 50  0000 C CNN
@@
 AR Path="/5DCE035A/5DDA1AFF" Ref="C?"  Part="1"
 F 0 "C6" V 12150 4075 50  0000 L CNN
-F 1 "22pF" V 11975 3950 50  0000 L CNN
+F 1 "1nF get rid of shitty high pitch noise" V 11975 3950 50  0000 L CNN
 F 2 "4ms_Capacitor:C_0603" H 12100 4025 50  0001 C CNN
 F 3 "" H 12100 4025 50  0000 C CNN
