File: tests/test/2DCO-2PI.kicad_pcb (KiCad board)
At the start: 2 copper layers, 300 x 110.2 mm, 162 parts, among them J7 OUTPUT

Commit message: created new layouts that seems interesting
Parts:
- removed the VR? at (138.9, 79.6)
- removed the VR? at (179.4, 79.6)
- removed the VR? at (148.0, 99.1)
- removed the VR? at (170.2, 98.8)
- removed the VR? at (159.2, 79.7)
- removed the VR? at (171.6, 43.5)
- removed the VR? at (148.9, 44.0)
- added VR?: 100k, 4ms_Potentiometer:Pot_9mm_Knurl_NoDet, F.Cu at (221.7, 27.6)
- added VR?: 100k, 4ms_Potentiometer:Pot_9mm_Knurl_NoDet, F.Cu at (204.9, 27.6)
- added VR?: 100k, 4ms_Potentiometer:Pot_9mm_Knurl_NoDet, F.Cu at (238.8, 27.4)
- moved 16mm 216.4 mm to (207.8, 68.0)
- moved 16mm 216.4 mm to (235.9, 67.6)
- moved 16mm 216.4 mm to (178.8, 67.6)
- moved 16mm 216.4 mm to (235.6, 93.4)
- moved 16mm 216.4 mm to (208.2, 92.7)
- moved 16mm 216.4 mm to (151.3, 92.7)
- moved 16mm 216.4 mm to (151.7, 67.3)
- moved 16mm 216.4 mm to (179.1, 92.7)
- moved VR? 216.4 mm to (235.3, 49.2)
- moved VR? 216.4 mm to (206.8, 49.2)
- moved VR? 216.4 mm to (178.4, 49.2)
- moved VR? 216.4 mm to (151.3, 48.9)
- moved POT 84.3 mm to (219.0, 6.94)
- moved REF** 84.3 mm to (209.6, 15.2)
- moved REF** 84.3 mm to (224.1, 15.3)
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Other:
- board text added: "CH 2 DCO"
- board text added: "CH 3 & 4 - Channels used for external patching? Maybe just PI functions?"
- board text removed: "CH 3 & 4 PI CIRCUITS GENERATE GATES AND ENVELOPES"
- board text removed: "CH2 DCO"
