File: tests/test/3CH-1GATE.kicad_pcb (KiCad board)
At the start: 2 copper layers, 300 x 110.2 mm, 162 parts, among them J7 OUTPUT

Commit message: created new layouts that seems interesting
Parts:
- removed the 16mm at (430.0, -28.2)
- removed the 16mm at (401.9, -27.9)
- removed the 16mm at (372.8, -28.2)
- removed the 16mm at (345.7, -28.5)
- removed the 16mm at (429.7, -2.43)
- removed the 16mm at (402.2, -3.10)
- removed the 16mm at (373.2, -3.10)
- removed the 16mm at (288.9, 88.2)
- removed the POT at (155.2, 62.0)
- removed the REF** at (155.3, 70.4)
- removed the REF** at (165.1, 70.5)
- removed the REF** at (145.7, 70.3)
- removed the REF** at (160.2, 70.4)
- removed the REF** at (150.4, 70.4)
- removed the REF** at (179.8, 62.1)
- removed the VR? at (138.9, 79.6)
- removed the VR? at (372.5, -46.6)
- removed the VR? at (345.4, -46.9)
- removed the VR? at (160.2, 26.3)
- removed the VR? at (179.4, 79.6)
- removed the VR? at (148.0, 99.1)
- removed the VR? at (170.2, 98.8)
- removed the VR? at (159.2, 79.7)
- removed the VR? at (171.6, 43.5)
- removed the VR? at (148.9, 44.0)
- removed the VR? at (429.3, -46.6)
- removed the VR? at (400.9, -46.6)
- moved 16mm 226.1 mm to (139.3, 89.8)
- moved 16mm 145.0 mm to (139.3, 59.8)
- moved 16mm 145.0 mm to (161.1, 72.4)
- moved 16mm 145.0 mm to (162.6, 38.5)
- moved POT 145.0 mm to (156.8, 7.65)
- moved REF** 145.0 mm to (156.9, 16.0)
- moved REF** 145.0 mm to (147.3, 15.9)
- moved REF** 145.0 mm to (187.2, 7.56)
- moved REF** 145.0 mm to (180.5, 7.56)
- moved REF** 145.0 mm to (161.8, 16.0)
- moved REF** 145.0 mm to (152.0, 16.0)
- moved VR? 145.0 mm to (178.5, 51.0)
- moved VR? 145.0 mm to (176.6, 84.0)
- moved 16mm 145.0 mm to (139.8, 29.8)
- moved REF** 145.0 mm to (166.7, 16.1)
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Other:
- board text added: "CH 2 DCO"
- board text added: "CH 3 AUX"
- board text added: "PATCHING IN AND OUT"
- board text added: "QCD ZONE"
- board text removed: "CH 3 & 4 PI CIRCUITS GENERATE GATES AND ENVELOPES"
- board text removed: "CH2 DCO"
- board text removed: "MASTER OUT"
- board text removed: "QCD/EXPANDER ZONE"
